Commit message: 重构硬件控制链并隔离 OpenDog 算法
拆分 MIT 与 OpenDog 硬件 runner，明确算法与硬件边界。

完善回零、目标限幅、速度配置和控制诊断，并同步更新模型配置、文档及测试。

File: ros2_ws/mit_robot/config/algorithm/dm1_opendog.urdf (robot description, URDF)
Before this commit: robot dm1_opendog, 18 links, 17 joints
Links:
- link LF_FOOT: mass 0.024302084286 -> 0.030285
- link LF_calf: mass 0.192776474180 -> 0.240236
- link LF_hip: mass 0.566780616299 -> 0.706316
- link LF_thigh: mass 0.784107130653 -> 0.977146
- link LH_FOOT: mass 0.024302084286 -> 0.030285
- link LH_calf: mass 0.192776474180 -> 0.240236
- link LH_hip: mass 0.566780616299 -> 0.706316
- link LH_thigh: mass 0.784107130653 -> 0.977146
- link RF_FOOT: mass 0.024302084286 -> 0.030285
- link RF_calf: mass 0.192776474180 -> 0.240236
- link RF_hip: mass 0.566780616299 -> 0.706316
- link RF_thigh: mass 0.784107130653 -> 0.977146
- link RH_FOOT: mass 0.024302084286 -> 0.030285
- link RH_calf: mass 0.192776474180 -> 0.240236
- link RH_hip: mass 0.566780616299 -> 0.706316
- link RH_thigh: mass 0.784107130653 -> 0.977146
- link base: mass 5.528134778326 -> 6.889103
